Commit message: 20190318

File: src/yumi_description/urdf/workspace.xacro (robot description, xacro)
@@ -19,14 +19,14 @@
       <visual>
         <geometry>
-          <box size="1.6 0.8 0.026"/>
+          <box size="0.8 0.8 0.026"/>
         </geometry>
-        <origin rpy="0 0 0" xyz="0 0 0"/>
+        <origin rpy="0 0 0" xyz="-0.4 0 0"/>
         <material name="Ivory"/>
       </visual>
       <collision>
         <geometry>
-          <box size="1.6 0.8 0.026"/>
+          <box size="0.8 0.8 0.026"/>
         </geometry>
-        <origin rpy="0 0 0" xyz="0 0 0"/>
+        <origin rpy="0 0 0" xyz="-0.4 0 0"/>
         <material name="Ivory"/>
       </collision>
@@ -68,5 +68,5 @@
           <mesh filename="package://yumi_description/meshes/base/IRB14000_BaseStand_Fixed.stl"/>
         </geometry>
-        <material name="Orange"/>
+        <material name="Ivory"/>
       </visual>
       <collision>
@@ -75,5 +75,5 @@
           <mesh filename="package://yumi_description/meshes/base/IRB14000_BaseStand_Fixed.stl"/>
         </geometry>
-        <material name="Orange"/>
+        <material name="Ivory"/>
       </collision>
     </link>
